File: pcb/rev.A/pc104_isa_adapter.kicad_sch (KiCad schematic)
At the start: 6 parts, among them J1 Bus_ISA_16bit, J2 PC104_16, J3 PC104, J4 Bus_ISA_16bit

Commit message: update pcb rev.A (final)
Parts:
- H1, H2, J1, J4: now left out of the parts list
Other:
- moved on the sheet: H1, H2, J1, J2, J4
